Commit message: ros2 controlのコントローラーのロードに成功

File: nr26_r2_sim/urdf/nr26_r2.urdf.xacro (robot description, xacro)
@@ -1,5 +1,13 @@
 <?xml version="1.0"?>
 <robot name="nr26_r2" xmlns:xacro="http://www.ros.org/wiki/xacro">
-  <!-- ===== パラメータ ===== -->
+  <ros2_control name="GazeboSimSystem" type="system">
+    <hardware>
+      <plugin>gz_ros2_control/GazeboSimSystem</plugin>
+    </hardware>
+    <joint name="wheel_fl_joint"><command_interface name="velocity"/><state_interface name="position"/><state_interface name="velocity"/></joint>
+    <joint name="wheel_fr_joint"><command_interface name="velocity"/><state_interface name="position"/><state_interface name="velocity"/></joint>
+    <joint name="wheel_rl_joint"><command_interface name="velocity"/><state_interface name="position"/><state_interface name="velocity"/></joint>
+    <joint name="wheel_rr_joint"><command_interface name="velocity"/><state_interface name="position"/><state_interface name="velocity"/></joint>
+  </ros2_control>
   <xacro:property name="wheel_radius" value="0.05"/>
   <xacro:property name="wheel_width"  value="0.02"/>
@@ -9,65 +17,62 @@
   <xacro:property name="base_height" value="0.08"/>
   <xacro:property name="base_mass"   value="10.0"/>
-  <!-- ===== base_link ===== -->
-  <link name="base_link">
+  <link name="base_link"/>
+  <link name="chassis">
     <visual>
-      <geometry>
-        <box size="${base_length} ${base_width} ${base_height}"/>
-      </geometry>
-      <material name="gray"/>
+      <geometry><box size="${base_length} ${base_width} ${base_height}"/></geometry>
+      <material name="gray"><color rgba="0.5 0.5 0.5 1.0"/></material>
     </visual>
     <collision>
-      <geometry>
-        <box size="${base_length} ${base_width} ${base_height}"/>
-      </geometry>
+      <geometry><box size="${base_length} ${base_width} ${base_height}"/></geometry>
     </collision>
     <inertial>
+      <origin xyz="0 0 0" rpy="0 0 0"/>
       <mass value="${base_mass}"/>
-      <origin xyz="0 0 0"/>
-      <inertia
-        ixx="0.2" ixy="0.0" ixz="0.0"
-        iyy="0.2" iyz="0.0"
-        izz="0.2"/>
+      <inertia ixx="0.1" ixy="0.0" ixz="0.0" iyy="0.1" iyz="0.0" izz="0.1"/>
     </inertial>
   </link>
-  <!-- ===== wheel macro ===== -->
+  <joint name="base_chassis_joint" type="fixed">
+    <parent link="base_link"/>
+    <child link="chassis"/>
+    <origin xyz="0 0 ${wheel_radius}" rpy="0 0 0"/>
+  </joint>
   <xacro:macro name="wheel" params="name x y">
     <link name="${name}">
       <visual>
-        <geometry>
-          <cylinder radius="${wheel_radius}" length="${wheel_width}"/>
-        </geometry>
-        <origin rpy="1.5708 0 0"/>
+        <origin rpy="${pi/2} 0 0" xyz="0 0 0"/>
+        <geometry><cylinder radius="${wheel_radius}" length="${wheel_width}"/></geometry>
+        <material name="black"><color rgba="0.1 0.1 0.1 1.0"/></material>
       </visual>
       <collision>
-        <geometry>
-          <cylinder radius="${wheel_radius}" length="${wheel_width}"/>
-        </geometry>
-        <origin rpy="1.5708 0 0"/>
+        <origin rpy="${pi/2} 0 0" xyz="0 0 0"/>
+        <geometry><cylinder radius="${wheel_radius}" length="${wheel_width}"/></geometry>
       </collision>
       <inertial>
+        <origin rpy="${pi/2} 0 0" xyz="0 0 0"/>
         <mass value="${wheel_mass}"/>
-        <inertia
-          ixx="0.001" ixy="0.0" ixz="0.0"
-          iyy="0.001" iyz="0.0"
-          izz="0.001"/>
+        <inertia ixx="0.001" ixy="0.0" ixz="0.0" iyy="0.001" iyz="0.0" izz="0.001"/>
       </inertial>
     </link>
     <joint name="${name}_joint" type="continuous">
-      <parent link="base_link"/>
+      <parent link="chassis"/>
       <child link="${name}"/>
-      <origin xyz="${x} ${y} -${base_height/2}" rpy="0 0 0"/>
+      <origin xyz="${x} ${y} -${wheel_radius}" rpy="0 0 0"/>
       <axis xyz="0 1 0"/>
     </joint>
-    <!-- Gazebo 摩擦設定（超重要） -->
     <gazebo reference="${name}">
-      <mu1>0.8</mu1>
-      <mu2>0.2</mu2>
+      <mu1 value="1.0"/>
+      <mu2 value="1.0"/>
+      <kp value="1000000.0" />
+      <kd value="1.0" />
     </gazebo>
   </xacro:macro>
-  <!-- ===== 4 wheels ===== -->
-  <xacro:wheel name="wheel_fl" x=" ${base_length/2}" y=" ${base_width/2}"/>
-  <xacro:wheel name="wheel_fr" x=" ${base_length/2}" y="-${base_width/2}"/>
-  <xacro:wheel name="wheel_rl" x="-${base_length/2}" y=" ${base_width/2}"/>
-  <xacro:wheel name="wheel_rr" x="-${base_length/2}" y="-${base_width/2}"/>
+  <xacro:wheel name="wheel_fl" x="0.15" y="0.17"/>
+  <xacro:wheel name="wheel_fr" x="0.15" y="-0.17"/>
+  <xacro:wheel name="wheel_rl" x="-0.15" y="0.17"/>
+  <xacro:wheel name="wheel_rr" x="-0.15" y="-0.17"/>
+  <gazebo>
+    <plugin name="gz_ros2_control::GazeboSimROS2ControlPlugin" filename="gz_ros2_control-system">
+      <parameters>$(find nr26_r2_sim)/config/nr26_r2_controllers.yaml</parameters>
+    </plugin>
+  </gazebo>
 </robot>
